File: hackclubMacropad.kicad_sch (KiCad schematic)
At the start: 21 parts, among them SW1 SW_Push, SW10 RotaryEncoder_Switch_MP, SW2 SW_Push, SW3 SW_Push, SW4 SW_Push, SW5 SW_Push, SW6 SW_Push, SW7 SW_Push, SW8 SW_Push, SW9 SW_Push, U1 MOUDLE-SEEEDUINO-XIAO

Commit message: added some 3d models to footprints
Parts:
- SW1, SW2, SW3, SW4, SW5, SW6, SW7, SW8, SW9: footprint Button_Switch_Keyboard:SW_Cherry_MX_1.00u_PCB -> footprints2:SW_Cherry_MX_1.00u_PCB
Changed lines of the file:
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@@
 			)
 		)
-		(property "Footprint" "Button_Switch_Keyboard:SW_Cherry_MX_1.00u_PCB"
+		(property "Footprint" "footprints2:SW_Cherry_MX_1.00u_PCB"
 			(at 167.64 96.52 0)
 			(effects
@@
 			)
 		)
-		(property "Footprint" "Button_Switch_Keyboard:SW_Cherry_MX_1.00u_PCB"
+		(property "Footprint" "footprints2:SW_Cherry_MX_1.00u_PCB"
 			(at 181.61 119.38 0)
 			(effects
@@
 			)
 		)
-		(property "Footprint" "Button_Switch_Keyboard:SW_Cherry_MX_1.00u_PCB"
+		(property "Footprint" "footprints2:SW_Cherry_MX_1.00u_PCB"
 			(at 167.64 119.38 0)
 			(effects
@@
 			)
 		)
-		(property "Footprint" "Button_Switch_Keyboard:SW_Cherry_MX_1.00u_PCB"
+		(property "Footprint" "footprints2:SW_Cherry_MX_1.00u_PCB"
 			(at 195.58 119.38 0)
 			(effects
@@
 			)
 		)
-		(property "Footprint" "Button_Switch_Keyboard:SW_Cherry_MX_1.00u_PCB"
+		(property "Footprint" "footprints2:SW_Cherry_MX_1.00u_PCB"
 			(at 181.61 96.52 0)
 			(effects
@@
 			)
 		)
-		(property "Footprint" "Button_Switch_Keyboard:SW_Cherry_MX_1.00u_PCB"
+		(property "Footprint" "footprints2:SW_Cherry_MX_1.00u_PCB"
 			(at 195.58 73.66 0)
 			(effects
@@
 			)
 		)
-		(property "Footprint" "Button_Switch_Keyboard:SW_Cherry_MX_1.00u_PCB"
+		(property "Footprint" "footprints2:SW_Cherry_MX_1.00u_PCB"
 			(at 195.58 96.52 0)
 			(effects
@@
 			)
 		)
-		(property "Footprint" "Button_Switch_Keyboard:SW_Cherry_MX_1.00u_PCB"
+		(property "Footprint" "footprints2:SW_Cherry_MX_1.00u_PCB"
 			(at 167.64 73.66 0)
 			(effects
@@
 			)
 		)
-		(property "Footprint" "Button_Switch_Keyboard:SW_Cherry_MX_1.00u_PCB"
+		(property "Footprint" "footprints2:SW_Cherry_MX_1.00u_PCB"
 			(at 181.61 73.66 0)
 			(effects
