File: pcb/hackclubMacropad.kicad_sch (KiCad schematic)
At the start: 21 parts, among them SW1 SW_Push, SW10 RotaryEncoder_Switch_MP, SW2 SW_Push, SW3 SW_Push, SW4 SW_Push, SW5 SW_Push, SW6 SW_Push, SW7 SW_Push, SW8 SW_Push, SW9 SW_Push, U1 MOUDLE-SEEEDUINO-XIAO

Commit message: commit autosaved files from pcb
Connections:
- net EC11MP: no longer names the net of U1.8 (PB09_A7_D7_RX)
- net EC11MP: no longer SW10.MP
Changed lines of the file:
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@@
-	(wire
-		(pts
-			(xy 156.21 121.92) (xy 165.1 121.92)
-		)
-		(stroke
-			(width 0)
-			(type default)
-		)
-	)
 	(wire
 		(pts
@@
 		(pts
 			(xy 223.52 161.29) (xy 237.49 161.29)
-		)
-		(stroke
-			(width 0)
-			(type default)
-		)
-	)
-	(wire
-		(pts
-			(xy 240.03 77.47) (xy 240.03 86.36)
 		)
 		(stroke
@@
 		)
 	)
-	(label "EC11MP"
-		(at 240.03 86.36 0)
-		(effects
-			(font
-				(size 1.27 1.27)
-			)
-			(justify left bottom)
-		)
-	)
 	(label "Row 0"
 		(at 106.68 106.68 0)
 		(effects
 			(font
-				(size 1.27 1.27)
-			)
-			(justify left bottom)
-		)
-	)
-	(label "EC11MP"
-		(at 165.1 121.92 0)
-		(effects
-			(font
